File: tiny-led-esp32.sch (KiCad schematic (older format))
At the start: 38 parts, among them J1 USB_B_Micro, U1 AMS1117-3.3, U2 ESP32-WROOM-32

Commit message: added mount holes, inner layers
Parts:
- added H1: GND, MountingHole:MountingHole_3.2mm_M3_Pad_Via, symbol Mechanical:MountingHole_Pad
- added H2: 5V, MountingHole:MountingHole_3.2mm_M3_Pad_Via, symbol Mechanical:MountingHole_Pad
Connections:
- net +5V: now also H2.1
- net GND: now also H1.1
Changed lines of the file:
@@
 Text GLabel 1200 3050 2    50   Input ~ 0
 TX
+$Comp
+L Mechanical:MountingHole_Pad H1
+U 1 1 6219DFBD
+P 1000 4900
+F 0 "H1" H 950 5100 50  0000 L CNN
+F 1 "GND" V 850 4850 50  0000 L CNN
+F 2 "MountingHole:MountingHole_3.2mm_M3_Pad_Via" H 1000 4900 50  0001 C CNN
+F 3 "~" H 1000 4900 50  0001 C CNN
+	1    1000 4900
+	1    0    0    -1
+$EndComp
+$Comp
+L Mechanical:MountingHole_Pad H2
+U 1 1 621A0917
+P 1300 4900
+F 0 "H2" H 1250 5100 50  0000 L CNN
+F 1 "5V" V 1150 4850 50  0000 L CNN
+F 2 "MountingHole:MountingHole_3.2mm_M3_Pad_Via" H 1300 4900 50  0001 C CNN
+F 3 "~" H 1300 4900 50  0001 C CNN
+	1    1300 4900
+	1    0    0    -1
+$EndComp
+Wire Wire Line
+	1000 5150 1000 5000
+Wire Wire Line
+	1300 5000 1300 5150
+$Comp
+L power:GND #PWR0101
+U 1 1 621B63E7
+P 1000 5150
+F 0 "#PWR0101" H 1000 4900 50  0001 C CNN
+F 1 "GND" H 1005 4977 50  0000 C CNN
+F 2 "" H 1000 5150 50  0001 C CNN
+F 3 "" H 1000 5150 50  0001 C CNN
+	1    1000 5150
+	1    0    0    -1
+$EndComp
+$Comp
+L power:+5V #PWR0102
+U 1 1 621EC70E
+P 1300 5150
+F 0 "#PWR0102" H 1300 5000 50  0001 C CNN
+F 1 "+5V" H 1315 5323 50  0000 C CNN
+F 2 "" H 1300 5150 50  0001 C CNN
+F 3 "" H 1300 5150 50  0001 C CNN
+	1    1300 5150
+	-1   0    0    1
+$EndComp
 $EndSCHEMATC

Commit message: finished with v0.1
Parts:
- added TP7: TestPoint, TestPoint:TestPoint_Pad_D2.5mm, symbol Connector:TestPoint
Connections:
- net IO0: now reaches U2.25 (IO0)
- net IO0: now also TP7.1
- net EN: now reaches R3.1, TP1.1, U2.3 (EN)
- no-connect marks 33 -> 32
Changed lines of the file:
@@
 	2250 1200 2250 1400
 Wire Wire Line
-	1300 1200 1300 1550
-Wire Wire Line
-	1300 1600 1650 1600
+	1300 1200 1300 1350
 $Comp
 L power:GND #PWR010
@@
 	0    -1   -1   0
 $EndComp
-Connection ~ 1300 1550
-Wire Wire Line
-	1300 1550 1300 1600
 NoConn ~ 1650 2800
 NoConn ~ 1650 2900
@@
 NoConn ~ 2850 2000
 NoConn ~ 2850 1800
-NoConn ~ 2850 1600
 NoConn ~ 1650 1800
 NoConn ~ 1650 1900
@@
 	-1   0    0    1
 $EndComp
+Text GLabel 1650 1600 0    50   Input ~ 0
+EN
+Text GLabel 1150 1350 0    50   Input ~ 0
+EN
+Wire Wire Line
+	1150 1350 1300 1350
+Connection ~ 1300 1350
+Wire Wire Line
+	1300 1350 1300 1550
+Text GLabel 2850 1600 2    50   Input ~ 0
+IO0
+$Comp
+L Connector:TestPoint TP7
+U 1 1 62245454
+P 1200 3650
+F 0 "TP7" V 1250 3700 50  0000 C CNN
+F 1 "TestPoint" V 1200 4000 50  0000 C CNN
+F 2 "TestPoint:TestPoint_Pad_D2.5mm" H 1400 3650 50  0001 C CNN
+F 3 "~" H 1400 3650 50  0001 C CNN
+	1    1200 3650
+	0    -1   -1   0
+$EndComp
+Text GLabel 1200 3650 2    50   Input ~ 0
+IO0
 $EndSCHEMATC
